File: Schaltpläne/Bewegungssensor/Schaltplan_Bewegungssensor/Schaltplan_Bewegungssensor.kicad_sch (KiCad schematic)
At the start: 8 parts, among them U1 LSM6DSOX_custom

Commit message: Add files via upload
Parts:
- removed TP_CS: TestPoint, symbol Connector:TestPoint
Connections:
- net +3.3V renamed 3.3V
